Commit message: updateModel

File: dogspace/src/spot/urdf/Dog.urdf (robot description, URDF)
Before this commit: robot dd_robot, 1 links, 0 joints
Links:
- added link right_h1; visual cylinder length=0.3 radius=0.02
- added link right_h2; visual cylinder length=0.3 radius=0.02
- added link right_j1; visual sphere radius=0.05
- added link right_j2; visual sphere radius=0.05
- added link right_knee1; visual sphere radius=0.05
- added link right_leg1; visual cylinder length=0.3 radius=0.02
Joints:
- added joint j_right_knee1: type continuous, parent right_h1, child right_knee1, origin xyz=0 0 -0.2 rpy=0 0 0, axis 0 1 0
- added joint j_right_leg1: type fixed, parent right_knee1, child right_leg1, origin xyz=0 0 -0.2 rpy=0 0 0, axis 0 1 0
- added joint joint_right_h1: type fixed, parent right_j1, child right_h1, origin xyz=0 0 -0.2 rpy=0 0 0, axis 0 1 0
- added joint joint_right_h2: type fixed, parent right_j2, child right_h2, origin xyz=0 0 -0.2 rpy=0 0 0, axis 0 1 0
- added joint joint_right_j1: type continuous, parent base_link, child right_j1, origin xyz=0.5 -0.30 0 rpy=0 0 0, axis 0 1 0
- added joint joint_right_j2: type continuous, parent base_link, child right_j2, origin xyz=-0.5 -0.30 0 rpy=0 0 0, axis 0 1 0

Commit message: hips_done

File: dogspace/src/spot/urdf/Dog.urdf (robot description, URDF)
Before this commit: robot dd_robot, 7 links, 6 joints
Links:
- removed link right_j1
- removed link right_j2
- removed link right_knee1
- removed link right_leg1
- added link left_h1; visual cylinder length=0.3 radius=0.02
- added link left_h2; visual cylinder length=0.3 radius=0.02
Joints:
- removed joint j_right_knee1
- removed joint j_right_leg1
- removed joint joint_right_j1
- removed joint joint_right_j2
- added joint joint_left_h1: type continuous, parent base_link, child left_h1, origin xyz=0.5 0.3 -0.2 rpy=0 0 0, axis 0 1 0
- added joint joint_left_h2: type continuous, parent base_link, child left_h2, origin xyz=-0.5 0.3 -0.2 rpy=0 0 0, axis 0 1 0
- joint joint_right_h1: origin xyz=0 0 -0.2 rpy=0 0 0 -> xyz=0.5 -0.3 -0.2 rpy=0 0 0; parent right_j1 -> base_link; type fixed -> continuous
- joint joint_right_h2: origin xyz=0 0 -0.2 rpy=0 0 0 -> xyz=-0.5 -0.3 -0.2 rpy=0 0 0; parent right_j2 -> base_link; type fixed -> continuous

Commit message: hip_with_joint

File: dogspace/src/spot/urdf/Dog.urdf (robot description, URDF)
Before this commit: robot dd_robot, 5 links, 4 joints
Links:
- link left_h1: geometry visual cylinder length=0.3 radius=0.02; visual sphere radius=0.05
- link left_h2: geometry visual cylinder length=0.3 radius=0.02; visual sphere radius=0.05
- link right_h1: geometry visual cylinder length=0.3 radius=0.02; visual sphere radius=0.05
- link right_h2: geometry visual cylinder length=0.3 radius=0.02; visual sphere radius=0.05

Commit message: Rviz_model

File: dogspace/src/spot/urdf/Dog.urdf (robot description, URDF)
Before this commit: robot dd_robot, 5 links, 4 joints
Links:
- added link left_k1; visual cylinder length=0.3 radius=0.02; visual sphere radius=0.05
- added link left_k2; visual cylinder length=0.3 radius=0.02; visual sphere radius=0.05
- added link right_k1; visual cylinder length=0.3 radius=0.02; visual sphere radius=0.05
- added link right_k2; visual cylinder length=0.3 radius=0.02; visual sphere radius=0.05
Joints:
- added joint joint_left_k1: type continuous, parent left_h1, child left_k1, origin xyz=0 0 -0.2 rpy=0 0 0, axis 0 1 0
- added joint joint_left_k2: type continuous, parent left_h2, child left_k2, origin xyz=0 0 -0.2 rpy=0 0 0, axis 0 1 0
- added joint joint_right_k1: type continuous, parent right_h1, child right_k1, origin xyz=0 0 -0.2 rpy=0 0 0, axis 0 1 0
- added joint joint_right_k2: type continuous, parent right_h2, child right_k2, origin xyz=0 0 -0.2 rpy=0 0 0, axis 0 1 0

Commit message: Adjust_pose

File: dogspace/src/spot/urdf/Dog.urdf (robot description, URDF)
Before this commit: robot dd_robot, 9 links, 8 joints
Links:
- link base_link: mass None -> 5
Joints:
- joint joint_left_h1: origin xyz=0.5 0.3 -0.2 rpy=0 0 0 -> xyz=0.5 0.3 0.4 rpy=0 0 0
- joint joint_left_h2: origin xyz=-0.5 0.3 -0.2 rpy=0 0 0 -> xyz=-0.5 0.3 0.4 rpy=0 0 0
- joint joint_right_h1: origin xyz=0.5 -0.3 -0.2 rpy=0 0 0 -> xyz=0.5 -0.3 0.4 rpy=0 0 0
- joint joint_right_h2: origin xyz=-0.5 -0.3 -0.2 rpy=0 0 0 -> xyz=-0.5 -0.3 0.4 rpy=0 0 0
