Commit message: working_camera

File: dogspace/src/spot/urdf/dog_gazebo.urdf (robot description, URDF)
Before this commit: robot dd_robot, 9 links, 8 joints
Links:
- added link camera_link, mass 5; collision box size=0.25 0.25 0.25; visual box size=0.25 0.25 0.25
Joints:
- added joint joint_camera: type continuous, parent base_link, child camera_link, origin xyz=0.5 0 0.8 rpy=0 0 0, axis 0 1 0

Commit message: camera_done

File: dogspace/src/spot/urdf/dog_gazebo.urdf (robot description, URDF)
Before this commit: robot dd_robot, 10 links, 9 joints
Joints:
- joint joint_camera: axis 0 1 0 -> 0 0 1
